File: board/kicad/tonnere/Microcontroller.kicad_sch (KiCad schematic)
At the start: 49 parts, among them J10 STM GPIO, J26 I2C, J9 STM SWD, Q2 2N7002, U10 74LVC1G17, U19 STM32F407ZGTx, U22 PCA9546APWR, U24 FSUSB42UMX-TP, Y1 8MHz, Y2 32.768KHz

Commit message: 0.60 (not final). Fix errata from 0.51. Added USB2 phy.
Parts:
- removed U24: FSUSB42UMX-TP, usb_switch:XQFN-10_L1.8-W1.4-P0.40-TL, symbol usb_switch:FSUSB42UMX-TP
- added C15, C18: 22pF, Capacitor_SMD:C_0603_1608Metric, symbol Device:C
- added C21, C22, C49: 4.7uF, Capacitor_SMD:C_0603_1608Metric, symbol Device:C
- added C30, C32, C40, C44: 0.1uF, Capacitor_SMD:C_0603_1608Metric, symbol Device:C
- added R37: 1m, Resistor_SMD:R_0603_1608Metric, symbol Device:R
- added R42: 12K 1%, Resistor_SMD:R_0603_1608Metric, symbol Device:R
- added R53: 820, Resistor_SMD:R_0603_1608Metric, symbol Device:R
- added R57: 0, Resistor_SMD:R_0603_1608Metric, symbol Device:R
- added SW2: USB HS/FS, dpdt:SW-SMD_MST22D18G2, symbol Switch:SW_Slide_DPDT
- added U17, U21: FSUSB42UMX-TP, usb_switch:XQFN-10_L1.8-W1.4-P0.40-TL, symbol usb_switch:FSUSB42UMX-TP
- added U20: USB3300-EZK, Package_DFN_QFN:QFN-32-1EP_5x5mm_P0.5mm_EP3.45x3.45mm, symbol Interface_USB:USB3300-EZK
- added U4: TPD4E02B04DQA, Package_SON:USON-10_2.5x1.0mm_P0.5mm, symbol Power_Protection:TPD4E02B04DQA
- added Y1: 24MHz, Crystal:Crystal_SMD_3225-4Pin_3.2x2.5mm, symbol Device:Crystal_GND24
- renumbered C15 to C16, C16 to C17, C24 to C20, C19 to C24, C20 to C25, C22 to C28, C27 to C34, C28 to C35, C29 to C36, C43 to C52, C46 to C55, C48 to C57, C51 to C60, C54 to C63, C55 to C64, C57 to C66, D2 to D6, J9 to J10, J26 to J27, J10 to J9, Q2 to Q3, R27 to R31, R33 to R39, R40 to R51, R46 to R54, R47 to R55, R51 to R60, R52 to R61, R53 to R62, R54 to R63, R68 to R77, R69 to R78, U10 to U11, U19 to U23, U22 to U26, Y1 to Y2, Y2 to Y3
Connections:
- net USART1.RTS is gone; now on an unnamed net: U23.75 (PB14)
- net +3V3: now also C30.1, C32.1, C40.1, C44.1, SW2.1 (A), U17.9 (VCC), U20.16 (VDD3.3), U20.25 (VDD3.3), U20.30 (VDD3.3), U20.31 (REG_EN), U20.6 (VDD3.3), U21.9 (VCC)
- net +V5_VBUS_FOR_DETECT: now also SW2.6 (C)
- net ESP.SGPIO: now also U23.100 (PA8); no longer U23.101 (PA9)
- net GND: now also D6.2 (A), C15.1, C18.1, C21.2, C22.2, C30.2, C32.2, C40.2, C44.2, C49.2, R42.2, R57.2, SW2.3 (C), U17.3 (GND), U17.8 (OE#), U20.1 (GND), U20.2 (GND), U20.33 (GND), U21.3 (GND), U21.8 (OE#), U4.3 (G), U4.8 (G), Y1.2, Y1.4; no longer D6.1 (K)
- net JOY.POT0: now also U23.18 (PF6); no longer U23.26 (PC0)
- net JOY.POT1: now also U23.19 (PF7); no longer U23.27 (PC1)
- net JOY.POT2: now also U23.20 (PF8); no longer U23.28 (PC2)
- net JOY.POT3: now also U23.21 (PF9); no longer U23.29 (PC3)
- net JOY2.POT4: now also U23.22 (PF10); no longer U23.34 (PA0)
- net JOY2.POT5: now also U23.27 (PC1); no longer U23.35 (PA1)
- net JOY2.POT6: now also U23.34 (PA0); no longer U23.40 (PA4)
- net JOY2.POT7: now also U23.35 (PA1); no longer U23.41 (PA5)
- net SPI.MOSI: now also U23.43 (PA7); no longer U23.135 (PB5)
- net STMAUD.ADC.R: now also U23.40 (PA4); no longer U23.37 (PA3)
- net STMAUD.ADC.SIO: now also U23.44 (PC4); no longer U23.43 (PA7)
- net USART1.RX: now also U23.102 (PA10); no longer U23.70 (PB11)
- net USART1.TX: now also U23.101 (PA9); no longer U23.69 (PB10)
- net USB.DM: now also U21.2 (D-)
- net USB.DP: now also U21.1 (D+)
- net at C20.2, Q3.1 (G), R51.1: now also D6.1 (K); no longer D6.2 (A)
- net STMUSB.DM1: now reaches R77.2
- net STMUSB.DM1: now also U17.4 (HSD1-), U21.6 (HSD2-)
- net at U23.1 (PE2): now also J9.7 (Pin_7)
- net at U23.110 (PA15): now also J9.6 (Pin_6)
- net at J9.5 (Pin_5): now also U23.76 (PB15); no longer U23.20 (PF8)
- net at J9.4 (Pin_4): no longer U23.21 (PF9)
- net at J9.3 (Pin_3): now also U23.49 (PF11); no longer U23.22 (PF10)
- net USBPHY.D1: now reaches U23.46 (PB0)
- net USBPHY.D1: now also U20.23 (DATA1)
- net USBPHY.D2: now reaches U23.47 (PB1)
- net USBPHY.D2: now also U20.22 (DATA2)
- net STMUSB.DP1: now reaches R78.2
- net STMUSB.DP1: now also U17.5 (HSD1+), U21.7 (HSD2+)
- net at USB2.A7 (D1-), USB2.B7 (D2-): now also U17.2 (D-), U4.1 (IO1)
- net at USB2.A6 (D1+), USB2.B6 (D2+): now also U17.1 (D+), U4.2 (IO2)
- net USART1.CK renamed USBPHY.D5
- net USBPHY.D5: now also U20.19 (DATA5)
- net USART1.CTS renamed USBPHY.D6
- net USBPHY.D6: now also U20.18 (DATA6)
- new net: C18.2, R37.2, U20.28 (XI), Y1.1
- new net: C15.2, R37.1, U20.27 (XO), Y1.3
- new net: SW2.2 (B), U17.10 (SEL), U21.10 (SEL)
- new net: C49.1, R53.2, SW2.5 (B)
- new net: R42.1, U20.32 (RBIAS)
- new net: R53.1, U20.4 (VBUS)
- new net: R57.1, U20.9 (RESET)
- new net +5V: SW2.4 (A)
- new net 1V8: C21.1, U20.15 (VDD1.8), U20.26 (VDD1.8)
- new net 1VA8: C22.1, U20.29 (VDDA1.8)
- new net STMUSB.DM2: U17.6 (HSD2-), U20.8 (DM), U21.4 (HSD1-)
- new net STMUSB.DP2: U17.7 (HSD2+), U20.7 (DP), U21.5 (HSD1+)
- new net USBPHY.CLK: U20.14 (CLKOUT), U23.41 (PA5)
- new net USBPHY.D0: U20.24 (DATA0), U23.37 (PA3)
- new net USBPHY.D3: U20.21 (DATA3), U23.69 (PB10)
- new net USBPHY.D4: U20.20 (DATA4), U23.70 (PB11)
- new net USBPHY.D7: U20.17 (DATA7), U23.135 (PB5)
- new net USBPHY.DIR: U20.12 (DIR), U23.28 (PC2)
- new net USBPHY.NXT: U20.11 (NXT), U23.29 (PC3)
- new net USBPHY.STP: U20.13 (STP), U23.26 (PC0)
- no-connect marks 9 -> 5
Other:
- note added: "Automatic DFU mode on VBUS connect - sends 10ms reset pulse on NSRT on connect."
- note added: "H:D2, L:D1 So H=HS_EXT,LS_HUB L=LS_EXT,HS_HUB"
- note removed: "Rail bulk"
- moved on the sheet: D6, J9
