File: board/kicad/tonnere/Microcontroller.kicad_sch (KiCad schematic)
At the start: 67 parts, among them J10 STM SWD, J27 I2C, J9 STM GPIO, Q3 2N7002, SW2 USB HS/FS, U11 74LVC1G17, U17 FSUSB42UMX-TP, U20 USB3300-EZK, U21 FSUSB42UMX-TP, U23 STM32F407ZGTx, U26 PCA9546APWR, U4 TPD4E02B04DQA, Y1 24MHz, Y2 8MHz, Y3 32.768KHz

Commit message: Created 0.61 production files using jlcpcb kicad plugin
Parts:
- BT1: LCSC (none) -> C964752
- C10, C20, C30, C32, C34, C35, C36, C40, C44, C52, C55, C57, C64, C66: LCSC (none) -> C14663
- C15, C18: LCSC (none) -> C1653
- C16, C17: LCSC (none) -> C327125
- C21, C22, C49: LCSC (none) -> C19666
- C24, C25: LCSC (none) -> C1647
- C28: LCSC (none) -> C28323
- C60, C63: LCSC (none) -> C23630
- D6: LCSC (none) -> C2128
- FB1: LCSC (none) -> C1012
- J10: LCSC (none) -> C225480
- J27: LCSC (none) -> C225517
- J9: LCSC (none) -> C225482
- JP1: LCSC (none) -> C49257
- Q3: LCSC (none) -> C8545
- R31, R55, R60: LCSC (none) -> C25804
- R37, R39, R9: LCSC (none) -> C22935
- R4, R5: LCSC (none) -> C23186
- R42: LCSC (none) -> C22790
- R51: LCSC (none) -> C25803
- R53: LCSC (none) -> C23253
- R54, R7: LCSC (none) -> C21190
- R57: LCSC (none) -> C21189; now left out of the parts list
- R61, R77, R78: LCSC (none) -> C23345
- R62, R63: LCSC (none) -> C23162
- RN10, RN7: LCSC (none) -> C12008
- SW2: LCSC (none) -> C431544
- U11: LCSC (none) -> C7836
- U17, U21: LCSC (none) -> C42370490
- U20: LCSC (none) -> C108383
- U23: LCSC (none) -> C36869
- U26: LCSC (none) -> C400705
- U4: LCSC (none) -> C106794
- USB2: LCSC (none) -> C2689968
- Y1: LCSC (none) -> C5122304
- Y2: LCSC (none) -> C2924617
- Y3: LCSC (none) -> C32346
