File: board/kicad/tonnere/atariinterfaces.kicad_sch (KiCad schematic)
At the start: 70 parts, among them J17 FPGA GPIO, J22 Conn_01x04_Pin, J5 PBI, J7 Conn_01x01, J8 PBI Option, Q1 BCX51, U12 TPD8E003DQDR, U13 TPD8E003DQDR, U16 TPD8E003DQDR, U20 TPD8E003DQDR, U25 TPD8E003DQDR, U27 SN74CB3T16211DGVR, U29 SN74CB3T16211DGVR, U31 SN74CB3T16211DGVR, U33 SN74CB3T16211DGVR, U4 TPD8E003DQDR, U5 TPD8E003DQDR, U6 TPD8E003DQDR, U7 TPD8E003DQDR, U8 TPD8E003DQDR, U9 TPD8E003DQDR

Commit message: 0.60 (not final). Fix errata from 0.51. Added USB2 phy.
Parts:
- removed J22: Conn_01x04_Pin, Connector_PinHeader_2.54mm:PinHeader_1x04_P2.54mm_Vertical, symbol Connector:Conn_01x04_Pin
- added J24: CONSOL, Connector_PinHeader_2.54mm:PinHeader_1x05_P2.54mm_Vertical, symbol Connector:Conn_01x05_Pin
- renumbered C33 to C38, C36 to C43, C47 to C56, C49 to C58, C59 to C71, C65 to C77, C68 to C81, C70 to C86, C75 to C92, C78 to C97, J15 to J16, J17 to J18, J5 to J6, R85 to R100, R20 to R24, R24 to R28, R26 to R30, R29 to R33, R30 to R34, R31 to R36, R32 to R38, R42 to R49, R44 to R50, R49 to R58, R58 to R67, R59 to R68, R63 to R72, R80 to R94, R83 to R98, U9 to U10, U12 to U13, U13 to U14, U16 to U18, U20 to U24, U25 to U28, U27 to U30, U29 to U32, U31 to U35, U33 to U37, U4 to U5, U5 to U6, U6 to U7, U7 to U8, U8 to U9
Connections:
- net CONSOL_EXT.OPTION: now also J24.4 (Pin_4)
- net CONSOL_EXT.SELECT: now also J24.3 (Pin_3)
- net CONSOL_EXT.START: now also J24.2 (Pin_2)
- net GND: now also J24.1 (Pin_1)
- net SIO.MOTOR: now also U35.21 (2A5); no longer R33.2, R34.1
- net SIO_EXT.MOTOR: now reaches U35.36 (2B5)
- net SIO_EXT.MOTOR: now also R33.2, R34.1
- net CONSOL_EXT.RESET: now reaches U35.37 (2B4)
- net CONSOL_EXT.RESET: now also J24.5 (Pin_5)
- no-connect marks 31 -> 28
