File: board/kicad/tonnere/atariinterfaces.kicad_sch (KiCad schematic)
At the start: 70 parts, among them J18 FPGA GPIO, J24 CONSOL, J6 PBI, J7 Conn_01x01, J8 PBI Option, Q1 BCX51, U10 TPD8E003DQDR, U13 TPD8E003DQDR, U14 TPD8E003DQDR, U18 TPD8E003DQDR, U24 TPD8E003DQDR, U28 TPD8E003DQDR, U30 SN74CB3T16211DGVR, U32 SN74CB3T16211DGVR, U35 SN74CB3T16211DGVR, U37 SN74CB3T16211DGVR, U5 TPD8E003DQDR, U6 TPD8E003DQDR, U7 TPD8E003DQDR, U8 TPD8E003DQDR, U9 TPD8E003DQDR

Commit message: Created 0.61 production files using jlcpcb kicad plugin
Parts:
- C11, C13, C38, C43, C56, C58, C71, C77: LCSC (none) -> C1622
- C5: LCSC (none) -> C883598
- C81, C86, C92, C97: LCSC (none) -> C14663
- EDGE1: value ~ -> (none)
- F1, F3, F4, F5, F6: LCSC (none) -> C269152
- J11, J16: value ~ -> (none); LCSC (none) -> C5431655
- J13, J3: value ~ -> (none); now left out of the parts list
- J18: LCSC (none) -> C225482
- J24: LCSC (none) -> C225480
- J7: LCSC (none) -> C492400
- J8: LCSC (none) -> C225519
- Q1: LCSC (none) -> C475643
- R100, R11, R12, R15, R38, R58, R72: LCSC (none) -> C23162
- R13, R33, R34: LCSC (none) -> C13167
- R24, R28: LCSC (none) -> C25804
- R30, R36, R49, R50, R67, R68, R94, R98: LCSC (none) -> C21190
- RN11, RN3, RN4, RN5, RN6, RN9: LCSC (none) -> C1980
- U10, U13, U14, U18, U24, U28, U5, U6, U7, U8, U9: LCSC (none) -> C2867469
- U30, U32, U35, U37: LCSC (none) -> C2674751
