File: board/kicad/tonnere/audio.kicad_sch (KiCad schematic)
At the start: 40 parts, among them J1 PJ-325C5-G, J2 PJ-325C5-BL, U17 PCM5102A

Commit message: 0.60 (not final). Fix errata from 0.51. Added USB2 phy.
Parts:
- renumbered C82 to C102, C83 to C103, C18 to C23, C25 to C26, C21 to C27, C32 to C29, C26 to C33, C31 to C39, C38 to C46, C39 to C47, C40 to C48, C42 to C51, R95 to R115, R96 to R116, R16 to R20, R19 to R23, R21 to R25, R22 to R26, R23 to R27, R25 to R29, R41 to R48, R48 to R56, R50 to R59, U17 to U19
Changed lines of the file:
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@@
 		(dnp no)
 		(fields_autoplaced yes)
-		(property "Reference" "C39"
+		(property "Reference" "C47"
 			(at 259.08 34.2899 0)
 			(effects
@@
 			(project "tonnere"
 				(path "/eb8e239c-f2ec-4b57-8f5c-6c75d6b59ab3/604d5f35-37e8-463f-8a2a-7557cd751eb4"
-					(reference "C39")
+					(reference "C47")
 					(unit 1)
 				)
@@
 		(dnp no)
 		(fields_autoplaced yes)
-		(property "Reference" "C40"
+		(property "Reference" "C48"
 			(at 241.3 34.2899 0)
 			(effects
@@
 			(project "tonnere"
 				(path "/eb8e239c-f2ec-4b57-8f5c-6c75d6b59ab3/604d5f35-37e8-463f-8a2a-7557cd751eb4"
-					(reference "C40")
+					(reference "C48")
 					(unit 1)
 				)
@@
 		(on_board yes)
 		(dnp no)
-		(property "Reference" "C31"
+		(property "Reference" "C39"
 			(at 129.54 46.228 0)
 			(effects
@@
 			(project "tonnere"
 				(path "/eb8e239c-f2ec-4b57-8f5c-6c75d6b59ab3/604d5f35-37e8-463f-8a2a-7557cd751eb4"
-					(reference "C31")
+					(reference "C39")
 					(unit 1)
 				)
@@
 		(on_board yes)
 		(dnp no)
-		(property "Reference" "R50"
+		(property "Reference" "R59"
 			(at 90.17 92.71 90)
 			(effects
@@
 			(project "tonnere"
 				(path "/eb8e239c-f2ec-4b57-8f5c-6c75d6b59ab3/604d5f35-37e8-463f-8a2a-7557cd751eb4"
-					(reference "R50")
+					(reference "R59")
 					(unit 1)
 				)
@@
 		(dnp no)
 		(fields_autoplaced yes)
-		(property "Reference" "R22"
+		(property "Reference" "R26"
 			(at 157.48 115.57 90)
 			(effects
@@
 			(project "tonnere"
 				(path "/eb8e239c-f2ec-4b57-8f5c-6c75d6b59ab3/604d5f35-37e8-463f-8a2a-7557cd751eb4"
-					(reference "R22")
+					(reference "R26")
 					(unit 1)
 				)
@@
 		(on_board yes)
 		(dnp no)
-		(property "Reference" "R41"
+		(property "Reference" "R48"
 			(at 89.916 87.63 90)
 			(effects
@@
 			(project "tonnere"
 				(path "/eb8e239c-f2ec-4b57-8f5c-6c75d6b59ab3/604d5f35-37e8-463f-8a2a-7557cd751eb4"
-					(reference "R41")
+					(reference "R48")
 					(unit 1)
 				)
@@
 		(on_board yes)
 		(dnp no)
-		(property "Reference" "C83"
+		(property "Reference" "C103"
 			(at 78.232 118.872 90)
 			(effects
@@
 			(project "tonnere"
 				(path "/eb8e239c-f2ec-4b57-8f5c-6c75d6b59ab3/604d5f35-37e8-463f-8a2a-7557cd751eb4"
-					(reference "C83")
+					(reference "C103")
 					(unit 1)
 				)
@@
 		(dnp no)
 		(fields_autoplaced yes)
-		(property "Reference" "C25"
+		(property "Reference" "C26"
 			(at 219.71 34.2899 0)
 			(effects
@@
 			(project "tonnere"
 				(path "/eb8e239c-f2ec-4b57-8f5c-6c75d6b59ab3/604d5f35-37e8-463f-8a2a-7557cd751eb4"
-					(reference "C25")
+					(reference "C26")
 					(unit 1)
 				)
@@
 		(dnp no)
 		(fields_autoplaced yes)
-		(property "Reference" "R21"
+		(property "Reference" "R25"
 			(at 157.48 124.46 90)
 			(effects
@@
 			(project "tonnere"
 				(path "/eb8e239c-f2ec-4b57-8f5c-6c75d6b59ab3/604d5f35-37e8-463f-8a2a-7557cd751eb4"
-					(reference "R21")
+					(reference "R25")
 					(unit 1)
 				)
@@
 		(dnp no)
 		(fields_autoplaced yes)
-		(property "Reference" "U17"
+		(property "Reference" "U19"
 			(at 111.3633 21.59 0)
 			(effects
@@
 			(project ""
 				(path "/eb8e239c-f2ec-4b57-8f5c-6c75d6b59ab3/604d5f35-37e8-463f-8a2a-7557cd751eb4"
-					(reference "U17")
+					(reference "U19")
 					(unit 1)
 				)
@@
 		(dnp no)
 		(fields_autoplaced yes)
-		(property "Reference" "R25"
+		(property "Reference" "R29"
 			(at 222.25 123.1899 0)
 			(effects
@@
 			(project "tonnere"
 				(path "/eb8e239c-f2ec-4b57-8f5c-6c75d6b59ab3/604d5f35-37e8-463f-8a2a-7557cd751eb4"
-					(reference "R25")
+					(reference "R29")
 					(unit 1)
 				)
@@
 		(on_board yes)
 		(dnp no)
-		(property "Reference" "C38"
+		(property "Reference" "C46"
 			(at 71.882 107.188 90)
 			(effects
@@
 			(project "tonnere"
 				(path "/eb8e239c-f2ec-4b57-8f5c-6c75d6b59ab3/604d5f35-37e8-463f-8a2a-7557cd751eb4"
-					(reference "C38")
+					(reference "C46")
 					(unit 1)
 				)
@@
 		(on_board yes)
 		(dnp no)
-		(property "Reference" "R96"
+		(property "Reference" "R116"
 			(at 64.516 148.844 0)
 			(effects
@@
 			(project "tonnere"
 				(path "/eb8e239c-f2ec-4b57-8f5c-6c75d6b59ab3/604d5f35-37e8-463f-8a2a-7557cd751eb4"
-					(reference "R96")
+					(reference "R116")
 					(unit 1)
 				)
@@
 		(on_board yes)
 		(dnp no)
-		(property "Reference" "C26"
+		(property "Reference" "C33"
 			(at 66.802 107.188 90)
 			(effects
@@
 			(project "tonnere"
 				(path "/eb8e239c-f2ec-4b57-8f5c-6c75d6b59ab3/604d5f35-37e8-463f-8a2a-7557cd751eb4"
-					(reference "C26")
+					(reference "C33")
 					(unit 1)
 				)
@@
 		(on_board yes)
 		(dnp no)
-		(property "Reference" "R48"
+		(property "Reference" "R56"
 			(at 90.17 90.17 90)
 			(effects
@@
 			(project "tonnere"
 				(path "/eb8e239c-f2ec-4b57-8f5c-6c75d6b59ab3/604d5f35-37e8-463f-8a2a-7557cd751eb4"
-					(reference "R48")
+					(reference "R56")
 					(unit 1)
 				)
@@
 		(dnp no)
 		(fields_autoplaced yes)
-		(property "Reference" "C21"
+		(property "Reference" "C27"
 			(at 128.27 36.8299 0)
 			(effects
@@
 			(project "tonnere"
 				(path "/eb8e239c-f2ec-4b57-8f5c-6c75d6b59ab3/604d5f35-37e8-463f-8a2a-7557cd751eb4"
-					(reference "C21")
+					(reference "C27")
 					(unit 1)
 				)
@@
 		(on_board yes)
 		(dnp no)
-		(property "Reference" "C42"
+		(property "Reference" "C51"
 			(at 76.962 107.188 90)
 			(effects
@@
 			(project "tonnere"
 				(path "/eb8e239c-f2ec-4b57-8f5c-6c75d6b59ab3/604d5f35-37e8-463f-8a2a-7557cd751eb4"
-					(reference "C42")
+					(reference "C51")
 					(unit 1)
 				)
@@
 		(on_board yes)
 		(dnp no)
-		(property "Reference" "R95"
+		(property "Reference" "R115"
 			(at 73.914 123.19 90)
 			(effects
@@
 			(project "tonnere"
 				(path "/eb8e239c-f2ec-4b57-8f5c-6c75d6b59ab3/604d5f35-37e8-463f-8a2a-7557cd751eb4"
-					(reference "R95")
+					(reference "R115")
 					(unit 1)
 				)
@@
 		(dnp no)
 		(fields_autoplaced yes)
-		(property "Reference" "R23"
+		(property "Reference" "R27"
 			(at 222.25 102.8699 0)
 			(effects
@@
 			(project "tonnere"
 				(path "/eb8e239c-f2ec-4b57-8f5c-6c75d6b59ab3/604d5f35-37e8-463f-8a2a-7557cd751eb4"
-					(reference "R23")
+					(reference "R27")
 					(unit 1)
 				)
@@
 		(on_board yes)
 		(dnp no)
-		(property "Reference" "C18"
+		(property "Reference" "C23"
 			(at 119.634 53.848 0)
 			(effects
@@
 			(project "tonnere"
 				(path "/eb8e239c-f2ec-4b57-8f5c-6c75d6b59ab3/604d5f35-37e8-463f-8a2a-7557cd751eb4"
-					(reference "C18")
+					(reference "C23")
 					(unit 1)
 				)
@@
 		(dnp no)
 		(fields_autoplaced yes)
-		(property "Reference" "R16"
+		(property "Reference" "R20"
 			(at 157.48 97.79 90)
 			(effects
@@
 			(project "tonnere"
 				(path "/eb8e239c-f2ec-4b57-8f5c-6c75d6b59ab3/604d5f35-37e8-463f-8a2a-7557cd751eb4"
-					(reference "R16")
+					(reference "R20")
 					(unit 1)
 				)
@@
 		(on_board yes)
 		(dnp no)
-		(property "Reference" "C32"
+		(property "Reference" "C29"
 			(at 61.722 107.188 90)
 			(effects
@@
 			(project "tonnere"
 				(path "/eb8e239c-f2ec-4b57-8f5c-6c75d6b59ab3/604d5f35-37e8-463f-8a2a-7557cd751eb4"
-					(reference "C32")
+					(reference "C29")
 					(unit 1)
 				)
@@
 		(on_board yes)
 		(dnp no)
-		(property "Reference" "R19"
+		(property "Reference" "R23"
 			(at 76.708 148.844 0)
 			(effects
@@
 			(project "tonnere"
 				(path "/eb8e239c-f2ec-4b57-8f5c-6c75d6b59ab3/604d5f35-37e8-463f-8a2a-7557cd751eb4"
-					(reference "R19")
+					(reference "R23")
 					(unit 1)
 				)
@@
 		(on_board yes)
 		(dnp no)
-		(property "Reference" "C82"
+		(property "Reference" "C102"
 			(at 78.232 129.032 90)
 			(effects
@@
 			(project "tonnere"
 				(path "/eb8e239c-f2ec-4b57-8f5c-6c75d6b59ab3/604d5f35-37e8-463f-8a2a-7557cd751eb4"
-					(reference "C82")
+					(reference "C102")
 					(unit 1)
 				)
