File: board/kicad/tonnere/audio.kicad_sch (KiCad schematic)
At the start: 41 parts, among them J28 JA23331-HA6Q-4F, U19 PCM5102A, U48 PLT237/T10WH

Commit message: Created 0.61 production files using jlcpcb kicad plugin
Parts:
- C1, C102, C103, C23, C27, C4, C6: LCSC (none) -> C23630
- C126, C26, C39, C48, C8: LCSC (none) -> C14663
- C2, C3: LCSC (none) -> C1604
- C29, C33, C46, C51: LCSC (none) -> C53987
- C47, C9: LCSC (none) -> C15850
- FB2: LCSC (none) -> C1012
- R1, R116, R23, R8: LCSC (none) -> C22935
- R10, R20, R25, R26: LCSC (none) -> C25819
- R115, R43, R48, R56, R59: LCSC (none) -> C21190
- R2, R6: LCSC (none) -> C23179
- R27, R29: LCSC (none) -> C25804
- U19: LCSC (none) -> C107671
