File: board/kicad/tonnere/cycloneve.kicad_sch (KiCad schematic)
At the start: 54 parts, among them J14 SPI CFG, J16 SPI SEL, J21 FPGA JTAG, U23 M25PX32-VMW, U26 M25PX32-VMW, U30 10CL040f484, Y3 25MHz, Y4 Si5351A-B-GT, Y5 ASE-27MHz, Y6 25MHz, Y7 Si5351A-B-GT

Commit message: 0.60 (not final). Fix errata from 0.51. Added USB2 phy.
Parts:
- renumbered C81 to C101, C90 to C113, C93 to C116, C56 to C65, C58 to C70, C60 to C72, C61 to C73, C62 to C74, C63 to C75, C64 to C76, C66 to C78, C69 to C83, C71 to C88, C72 to C90, C73 to C91, C77 to C96, C79 to C99, J14 to J15, J16 to J17, J21 to J22, R86 to R101, R87 to R102, R89 to R104, R97 to R118, R98 to R120, R100 to R123, R103 to R126, R106 to R129, R107 to R130, R108 to R131, R60 to R69, R61 to R70, R62 to R71, R65 to R73, R64 to R74, R66 to R75, R67 to R76, R72 to R84, R77 to R92, R78 to R93, R81 to R95, R82 to R96, R79 to R97, R84 to R99, U23 to U27, U26 to U29, U30 to U33, Y3 to Y4, Y4 to Y5, Y5 to Y6, Y6 to Y7, Y7 to Y8
Connections:
- net VDAC.G is gone; now on net GND: U33.G2 (CLK0)
- net GND: now also U33.AA12 (CLK13), U33.AB12 (CLK12)
- net SRAM2.A1: now also U33.AB14 (IO); no longer U33.AA14 (IO)
- net SRAM2.A10: now also U33.AB18 (IO); no longer U33.AA18 (IO)
- net SRAM2.A11: now also U33.Y17 (IO); no longer U33.W17 (IO)
- net SRAM2.A12: now also U33.AA18 (IO); no longer U33.AB18 (IO)
- net SRAM2.A13: now also U33.W17 (IO); no longer U33.Y17 (IO)
- net SRAM2.A3: now also U33.AA14 (IO); no longer U33.W14 (IO)
- net SRAM2.A4: now also U33.R14 (IO); no longer U33.AB14 (IO)
- net SRAM2.D10: now also U33.Y13 (IO); no longer U33.AB12 (CLK12)
- net SRAM2.D4: now also U33.AB15 (IO); no longer U33.AA15 (IO)
- net SRAM2.D6: now also U33.AA15 (IO); no longer U33.AB15 (IO)
- net SRAM2.D7: now also U33.AB16 (IO); no longer U33.AA16 (IO)
- net SRAM2.D8: now also U33.AA13 (IO); no longer U33.Y13 (IO)
- net SRAM2.D9: now also U33.T13 (IO); no longer U33.AA12 (CLK13)
- net SRAM2.OE_N: now also U33.AB13 (IO); no longer U33.AA13 (IO)
- net SRAM2.UB_N: now also U33.W14 (IO); no longer U33.AB13 (IO)
- net SRAM2.W_N: now also U33.AA16 (IO); no longer U33.AB16 (IO)
- net VDAC.R1: now reaches U33.E3 (DIFFIO_L4n)
- net VDAC.R2: now reaches U33.E4 (DIFFIO_L4p)
- net VDAC.G0: now reaches U33.F1 (DIFFIO_L12n)
- net VDAC.G1: now reaches U33.F2 (DIFFIO_L12p)
- net VDAC.G2: now reaches U33.G3 (DIFFIO_L1n)
- net VDAC.B0: now reaches U33.H1 (DIFFIO_L23n)
- net VDAC.B1: now reaches U33.H2 (DIFFIO_L23p)
- net VDAC.B renamed VDAC.B2
- net VDAC.R renamed VDAC.R0
- no-connect marks 44 -> 35
