File: board/kicad/tonnere/cycloneve.kicad_sch (KiCad schematic)
At the start: 54 parts, among them J15 SPI CFG, J17 SPI SEL, J22 FPGA JTAG, U27 M25PX32-VMW, U29 M25PX32-VMW, U33 10CL040f484, Y4 25MHz, Y5 Si5351A-B-GT, Y6 ASE-27MHz, Y7 25MHz, Y8 Si5351A-B-GT

Commit message: Created 0.61 production files using jlcpcb kicad plugin
Parts:
- C101, C116, C65, C70, C72, C73, C74, C75, C76, C78, C83, C88, C90, C91, C96, C99: LCSC (none) -> C14663
- C113: LCSC (none) -> C57112
- FB5, FB7: LCSC (none) -> C1012
- J15: LCSC (none) -> C225518
- J17: LCSC (none) -> C49257
- J22: LCSC (none) -> C5665
- R101, R102, R118, R69, R70, R73, R74, R75, R99: LCSC (none) -> C25804
- R104: LCSC (none) -> C21190
- R120, R123, R126, R130, R71, R76, R84, R95, R96: LCSC (none) -> C23345
- R129, R131, R92, R93: LCSC (none) -> C23162
- R97: LCSC (none) -> C13167
- U27: LCSC (none) -> C2944643
- U29: LCSC (none) -> C2944643; now in the parts list
- U33: LCSC (none) -> C1521940
- Y4, Y7: LCSC (none) -> C337661
- Y5, Y8: LCSC (none) -> C504891
- Y6: LCSC (none) -> C37635418
Connections:
- net unconnected-(U33G-IO-PadG13): now reaches U33.G13 (IO)
- net unconnected-(U33G-IO-PadG14): now reaches U33.G14 (IO)
- net unconnected-(U33G-IO-PadG15): now reaches U33.G15 (IO)
- net unconnected-(U33G-IO-PadH15): now reaches U33.H15 (IO)
- net Net-(U33J-CLK6): now reaches R123.2, U33.T21 (CLK6)
- net unconnected-(U33E-IO-PadM16): now reaches U33.M16 (IO)
- net unconnected-(U33E-IO-PadP15): now reaches U33.P15 (IO)
- net unconnected-(U33E-IO-PadP16): now reaches U33.P16 (IO)
- net Net-(U33J-CLK14): now reaches R95.2, U33.AB11 (CLK14)
- net Net-(U33J-CLK2): now reaches R84.2, U33.T2 (CLK2)
- net unconnected-(U33H-IO-PadG10): now reaches U33.G10 (IO)
- net unconnected-(U33H-IO-PadG7): now reaches U33.G7 (IO)
- net unconnected-(U33H-IO-PadH10): now reaches U33.H10 (IO)
- net Net-(U33J-CLK5): now reaches R126.2, U33.G22 (CLK5)
- net unconnected-(U33C-IO-PadT10): now reaches U33.T10 (IO)
- net Net-(U33J-CLK8): now reaches R120.2, U33.A12 (CLK8)
- net Net-(U33J-CLK4): now reaches R130.2, U33.G21 (CLK4)
- net Net-(U33J-CLK3): now reaches R76.2, U33.T1 (CLK3)
- net unconnected-(U33B-IO-PadN7): now reaches U33.N7 (IO)
- net unconnected-(U33B-IO-PadP5): now reaches U33.P5 (IO)
- net unconnected-(U33B-IO-PadP6): now reaches U33.P6 (IO)
- net unconnected-(U33B-IO-PadU1): now reaches U33.U1 (IO)
- net unconnected-(U33B-IO-PadU2): now reaches U33.U2 (IO)
- net unconnected-(U33A-DIFFIO_L2n-PadB1): now reaches U33.B1 (DIFFIO_L2n)
- net unconnected-(U33A-DIFFIO_L2p-PadB2): now reaches U33.B2 (DIFFIO_L2p)
- net unconnected-(U33A-IO-PadH5): now reaches U33.H5 (IO)
- net unconnected-(U33A-DIFFIO_L9p-PadH6): now reaches U33.H6 (DIFFIO_L9p)
- net unconnected-(U33A-IO-PadH7): now reaches U33.H7 (IO)
- net unconnected-(U33A-DIFFIO_L14p-PadH8): now reaches U33.H8 (DIFFIO_L14p)
- net unconnected-(U33A-DIFFIO_L24n-PadJ1): now reaches U33.J1 (DIFFIO_L24n)
- net unconnected-(U33A-DIFFIO_L24p-PadJ2): now reaches U33.J2 (DIFFIO_L24p)
- net unconnected-(U33A-DIFFIO_L18n-PadJ5): now reaches U33.J5 (DIFFIO_L18n)
- net unconnected-(U33A-DIFFIO_L9n-PadJ6): now reaches U33.J6 (DIFFIO_L9n)
- net unconnected-(U33A-DIFFIO_L21p-PadJ7): now reaches U33.J7 (DIFFIO_L21p)
- net unconnected-(U33A-DIFFIO_L14n-PadJ8): now reaches U33.J8 (DIFFIO_L14n)
- net unconnected-(U33A-DIFFIO_L21n-PadK7): now reaches U33.K7 (DIFFIO_L21n)
- net unconnected-(U33A-DIFFIO_L20n-PadK8): now reaches U33.K8 (DIFFIO_L20n)
- net unconnected-(U33A-DIFFIO_L20p-PadL8): now reaches U33.L8 (DIFFIO_L20p)
