File: board/kicad/tonnere/power.kicad_sch (KiCad schematic)
At the start: 31 parts, among them SW1 SA-0-102-C04-0004-WP, U14 TPS62903RPJR, U15 TPS62903RPJR, U18 TPS62903RPJR

Commit message: 0.60 (not final). Fix errata from 0.51. Added USB2 phy.
Parts:
- added D2, D3, D4, D5: LED_RED, LED_SMD:LED_0805_2012Metric, symbol Device:LED
- added J12: Conn_01x05, Connector_PinHeader_2.54mm:PinHeader_1x05_P2.54mm_Vertical, symbol Connector_Generic:Conn_01x05
- added Q2: DMN2058U, Package_TO_SOT_SMD:SOT-23, symbol Transistor_FET:DMN2058U
- added R16: 1k, Resistor_SMD:R_0603_1608Metric, symbol Device:R
- added R17, R18, R19: 470, Resistor_SMD:R_0603_1608Metric, symbol Device:R
- added R35: 100k, Resistor_SMD:R_0603_1608Metric, symbol Device:R
- SW1: JLC_3DModel (none) -> 1b2c176f3639467abbcc028bfae2d8b5; JLC_3D_Size (none) -> 23.282 5.8
- renumbered C17 to C19, C23 to C31, C30 to C37, C34 to C41, C35 to C42, C37 to C45, C41 to C50, R17 to R21, R18 to R22, R28 to R32, R34 to R40, R35 to R41, R36 to R44, R37 to R45, R45 to R52, U14 to U15, U15 to U16, U18 to U22
Connections:
- net +1V2: now also J12.5 (Pin_5), Q2.1 (G), R35.1
- net +2V5: now also J12.4 (Pin_4), R18.1
- net +3V3: now also J12.3 (Pin_3), R17.1, R19.1
- net +5V: now also SW1.3, J12.2 (Pin_2), R16.1; no longer SW1.1
- net GND: now also D2.1 (K), D3.1 (K), D4.1 (K), J12.1 (Pin_1), Q2.2 (S), R35.2; no longer SW1.3
- new net: D5.2 (A), R19.2
- new net: D5.1 (K), Q2.3 (D)
- new net: D2.2 (A), R16.2
- new net: D4.2 (A), R18.2
- new net: D3.2 (A), R17.2
- no-connect marks 6 -> 7
