File: board/kicad/tonnere/power.kicad_sch (KiCad schematic)
At the start: 42 parts, among them J12 Conn_01x05, Q2 DMN2058U, SW1 SA-0-102-C04-0004-WP, U15 TPS62903RPJR, U16 TPS62903RPJR, U22 TPS62903RPJR

Commit message: Created 0.61 production files using jlcpcb kicad plugin
Parts:
- C12, C31, C42: LCSC (none) -> C57112
- C14, C37, C45: LCSC (none) -> C15850
- C19, C41, C50: LCSC (none) -> C45783
- C7: LCSC (none) -> C883598
- D2, D3, D4, D5: LCSC (none) -> C84256
- J12: LCSC (none) -> C225480
- L1, L2, L3: LCSC (none) -> C435392
- Q2: LCSC (none) -> C461001
- R16: LCSC (none) -> C21190
- R17, R18, R19: LCSC (none) -> C23179
- R21, R22: LCSC (none) -> C23186
- R32: LCSC (none) -> C2998122
- R35: LCSC (none) -> C25803
- R40: LCSC (none) -> C2933218
- R41, R52: LCSC (none) -> C49196678
- R44, R45: LCSC (none) -> C25819
- SW1: LCSC (none) -> C22449118
- U15, U16, U22: LCSC (none) -> C2866502
- USB1: LCSC (none) -> C2689968
