File: board/kicad/tonnere/esp32.kicad_sch (KiCad schematic)
At the start: 11 parts, among them J19 ESP PGM, J23 ESP JTAG, U40 ESP32-WROVER-E-N8R8

Commit message: Created 0.61 production files using jlcpcb kicad plugin
Parts:
- C115: LCSC (none) -> C14663
- C117: LCSC (none) -> C15850
- J19: LCSC (none) -> C225480
- J23: LCSC (none) -> C5665
- R103, R106, R108, R110, R113, R121: LCSC (none) -> C25804
- U40: LCSC (none) -> C529589
