File: board/kicad/tonnere/io_cards.kicad_sch (KiCad schematic)
At the start: 11 parts, among them U46 TPD4E02B04DQA, U47 TPD4E02B04DQA

Commit message: Created 0.61 production files using jlcpcb kicad plugin
Parts:
- C122, C54: value 120uF -> 100uF; LCSC (none) -> C883598
- C123, C53: LCSC (none) -> C14663
- Card1: LCSC (none) -> C164170
- Card2: LCSC (none) -> C125615
- RN12, RN13, RN8: LCSC (none) -> C102673
- U46, U47: LCSC (none) -> C106794
