File: board/kicad/tonnere/ram.kicad_sch (KiCad schematic)
At the start: 8 parts, among them U31 IS61WV204816BLL-10BLI, U36 IS61WV204816BLL-10BLI, U42 AS4C16M16SA

Commit message: Created 0.61 production files using jlcpcb kicad plugin
Parts:
- C108, C109, C79, C94: LCSC (none) -> C14663
- R112: LCSC (none) -> C23345
- U31: LCSC (none) -> C1349085
- U36: LCSC (none) -> C1348743
- U42: LCSC (none) -> C62246
