File: board/kicad/tonnere/tonnere.kicad_pcb (KiCad board)
At the start: 6 copper layers, 256.2 x 141.3 mm, 404 parts, among them J10 STM SWD, J12 Conn_01x05, J14 STM USART TTL, J15 SPI CFG, J17 SPI SEL, J18 FPGA GPIO, J19 ESP PGM, J20 USB_A, J21 73725-1180RLF, J22 FPGA JTAG, J23 ESP JTAG, J24 CONSOL, J25 73725-1180RLF, J26 73725-1180RLF, J27 I2C, J28 JA23331-HA6Q-4F, J4 DE15_Pins_HighDensity_Mountin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, J5 HDMI_A, J6 PBI, J7 Conn_01x01, J8 PBI Option, J9 STM GPIO, Q1 BCX51, Q2 DMN2058U, Q3 2N7002, SW1 SA-0-102-C04-0004-WP, SW2 USB HS/FS, U1 TPD4E02B04DQA, U10 TPD8E003DQDR, U11 74LVC1G17, U12 TPD4E02B04DQA, U13 TPD8E003DQDR, U14 TPD8E003DQDR, U15 TPS62903RPJR, U16 TPS62903RPJR, U17 FSUSB42UMX-TP, U18 TPD8E003DQDR, U19 PCM5102A, U2 TPD4E02B04DQA, U20 USB3300-EZK, U21 FSUSB42UMX-TP, U22 TPS62903RPJR, U23 STM32F407ZGTx, U24 TPD8E003DQDR, U25 THS7316DR, U26 PCA9546APWR, U27 M25PX32-VMW, U28 TPD8E003DQDR, U29 M25PX32-VMW, U3 TPD4E02B04DQA, U30 SN74CB3T16211DGVR, U31 IS61WV204816BLL-10BLI, U32 SN74CB3T16211DGVR, U33 10CL040f484, U34 AP2553AW6-7, U35 SN74CB3T16211DGVR, U36 IS61WV204816BLL-10BLI, U37 SN74CB3T16211DGVR, U38 AP2553AW6-7, U39 AP2553AW6-7, U4 TPD4E02B04DQA, U40 ESP32-WROVER-E-N8R8, U41 AP2553AW6-7, U42 AS4C16M16SA, U43 TPD4E02B04DQA, U44 USB2514B_Bi, U45 TPD4E02B04DQA, U46 TPD4E02B04DQA, U47 TPD4E02B04DQA, U48 PLT237/T10WH, U5 TPD8E003DQDR, U6 TPD8E003DQDR, U7 TPD8E003DQDR, U8 TPD8E003DQDR, U9 TPD8E003DQDR, Y1 24MHz, Y2 8MHz, Y3 32.768KHz, Y4 25MHz, Y5 Si5351A-B-GT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

Commit message: Created 0.61 production files using jlcpcb kicad plugin
Parts:
- C107, C122, C54, C80, C82, C85, C98: value 120uF -> 100uF
Connections:
- U33 pad B1: unconnected-(U33A-DIFFIO_L2n-PadB1) -> /FPGA/unconnected-(U33A-DIFFIO_L2n-PadB1)
- U33 pad B2: unconnected-(U33A-DIFFIO_L2p-PadB2) -> /FPGA/unconnected-(U33A-DIFFIO_L2p-PadB2)
- U33 pad G10: unconnected-(U33H-IO-PadG10) -> /FPGA/unconnected-(U33H-IO-PadG10)
- U33 pad G13: unconnected-(U33G-IO-PadG13) -> /FPGA/unconnected-(U33G-IO-PadG13)
- U33 pad G14: unconnected-(U33G-IO-PadG14) -> /FPGA/unconnected-(U33G-IO-PadG14)
- U33 pad G15: unconnected-(U33G-IO-PadG15) -> /FPGA/unconnected-(U33G-IO-PadG15)
- U33 pad G7: unconnected-(U33H-IO-PadG7) -> /FPGA/unconnected-(U33H-IO-PadG7)
- U33 pad H10: unconnected-(U33H-IO-PadH10) -> /FPGA/unconnected-(U33H-IO-PadH10)
- U33 pad H15: unconnected-(U33G-IO-PadH15) -> /FPGA/unconnected-(U33G-IO-PadH15)
- U33 pad H5: unconnected-(U33A-IO-PadH5) -> /FPGA/unconnected-(U33A-IO-PadH5)
- U33 pad H6: unconnected-(U33A-DIFFIO_L9p-PadH6) -> /FPGA/unconnected-(U33A-DIFFIO_L9p-PadH6)
- U33 pad H7: unconnected-(U33A-IO-PadH7) -> /FPGA/unconnected-(U33A-IO-PadH7)
- U33 pad H8: unconnected-(U33A-DIFFIO_L14p-PadH8) -> /FPGA/unconnected-(U33A-DIFFIO_L14p-PadH8)
- U33 pad J1: unconnected-(U33A-DIFFIO_L24n-PadJ1) -> /FPGA/unconnected-(U33A-DIFFIO_L24n-PadJ1)
- U33 pad J2: unconnected-(U33A-DIFFIO_L24p-PadJ2) -> /FPGA/unconnected-(U33A-DIFFIO_L24p-PadJ2)
- U33 pad J5: unconnected-(U33A-DIFFIO_L18n-PadJ5) -> /FPGA/unconnected-(U33A-DIFFIO_L18n-PadJ5)
- U33 pad J6: unconnected-(U33A-DIFFIO_L9n-PadJ6) -> /FPGA/unconnected-(U33A-DIFFIO_L9n-PadJ6)
- U33 pad J7: unconnected-(U33A-DIFFIO_L21p-PadJ7) -> /FPGA/unconnected-(U33A-DIFFIO_L21p-PadJ7)
- U33 pad J8: unconnected-(U33A-DIFFIO_L14n-PadJ8) -> /FPGA/unconnected-(U33A-DIFFIO_L14n-PadJ8)
- U33 pad K7: unconnected-(U33A-DIFFIO_L21n-PadK7) -> /FPGA/unconnected-(U33A-DIFFIO_L21n-PadK7)
- U33 pad K8: unconnected-(U33A-DIFFIO_L20n-PadK8) -> /FPGA/unconnected-(U33A-DIFFIO_L20n-PadK8)
- U33 pad L8: unconnected-(U33A-DIFFIO_L20p-PadL8) -> /FPGA/unconnected-(U33A-DIFFIO_L20p-PadL8)
- U33 pad M16: unconnected-(U33E-IO-PadM16) -> /FPGA/unconnected-(U33E-IO-PadM16)
- U33 pad N7: unconnected-(U33B-IO-PadN7) -> /FPGA/unconnected-(U33B-IO-PadN7)
- U33 pad P15: unconnected-(U33E-IO-PadP15) -> /FPGA/unconnected-(U33E-IO-PadP15)
- U33 pad P16: unconnected-(U33E-IO-PadP16) -> /FPGA/unconnected-(U33E-IO-PadP16)
- U33 pad P5: unconnected-(U33B-IO-PadP5) -> /FPGA/unconnected-(U33B-IO-PadP5)
- U33 pad P6: unconnected-(U33B-IO-PadP6) -> /FPGA/unconnected-(U33B-IO-PadP6)
- U33 pad T10: unconnected-(U33C-IO-PadT10) -> /FPGA/unconnected-(U33C-IO-PadT10)
- U33 pad U1: unconnected-(U33B-IO-PadU1) -> /FPGA/unconnected-(U33B-IO-PadU1)
- U33 pad U2: unconnected-(U33B-IO-PadU2) -> /FPGA/unconnected-(U33B-IO-PadU2)
