File: board/kicad/tonnere/usb.kicad_sch (KiCad schematic)
At the start: 51 parts, among them J20 USB_A, J21 73725-1180RLF, J25 73725-1180RLF, J26 73725-1180RLF, U34 AP2553AW6-7, U38 AP2553AW6-7, U39 AP2553AW6-7, U41 AP2553AW6-7, U43 TPD4E02B04DQA, U44 USB2514B_Bi, U45 TPD4E02B04DQA, Y9 24MHz

Commit message: Created 0.61 production files using jlcpcb kicad plugin
Parts:
- C100, C104, C105, C110, C112, C114, C118, C119, C120, C84, C87, C89, C93, C95: LCSC (none) -> C14663
- C106: LCSC (none) -> C28323
- C107, C80, C82, C85, C98: value 120uF -> 100uF; LCSC (none) -> C883598
- C111, C121: LCSC (none) -> C14663; now left out of the parts list
- C124, C125: LCSC (none) -> C1647
- FB6: LCSC (none) -> C1012
- J20: LCSC (none) -> C586225
- J21, J25, J26: LCSC (none) -> C26235
- R105, R109, R114, R119: LCSC (none) -> C4184
- R107, R111, R117, R122, R128: LCSC (none) -> C25804
- R124, R125, R127, R132: LCSC (none) -> C25803
- R133: LCSC (none) -> C22790
- U34, U38, U39, U41: LCSC (none) -> C441827
- U43, U45: LCSC (none) -> C106794
- U44: LCSC (none) -> C16251
- Y9: LCSC (none) -> C5122304
