File: board/kicad/tonnere/video.kicad_sch (KiCad schematic)
At the start: 38 parts, among them J4 DE15_Pins_HighDensity_Mountin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, J5 HDMI_A, U1 TPD4E02B04DQA, U12 TPD4E02B04DQA, U2 TPD4E02B04DQA, U25 THS7316DR, U3 TPD4E02B04DQA

Commit message: Created 0.61 production files using jlcpcb kicad plugin
Parts:
- C59: LCSC (none) -> C45783
- C61: LCSC (none) -> C15850
- C62: LCSC (none) -> C14663
- C67, C68, C69: LCSC (none) -> C1663
- D1: LCSC (none) -> C83329
- F2: LCSC (none) -> C3760613
- FB3, FB4: LCSC (none) -> C1012
- J4: LCSC (none) -> C7498158
- J5: LCSC (none) -> C138388
- R14, R3: LCSC (none) -> C23162
- R46, R47: LCSC (none) -> C22775
- R64, R65, R66: LCSC (none) -> C4275
- R79, R80, R81: LCSC (none) -> C543637
- R82, R86, R88: LCSC (none) -> C4109305
- R83, R89, R91: LCSC (none) -> C705739
- R85, R87, R90: LCSC (none) -> C705780
- RN1, RN2: LCSC (none) -> C1966
- U1, U12, U2, U3: LCSC (none) -> C106794
- U25: LCSC (none) -> C544774
