File: keyboard/key.kicad_sch (KiCad schematic)
At the start: 2 parts, among them SW10 MX

Commit message: Production file fixes for the keyboard PCB
Parts:
- SW10: FT Layer Override (none) -> bottom; FT Position Offset (none) -> 0.635,3.81; FT Rotation Offset (none) -> 180
Changed lines of the file:
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@@
+			)
+		)
+		(property "FT Layer Override" ""
+			(at 130.81 92.71 90)
+			(hide yes)
+			(show_name no)
+			(do_not_autoplace no)
+			(effects
+				(font
+					(size 1.27 1.27)
+				)
 			)
 		)
@@
 			(at 125.73 96.52 0)
 			(hide yes)
+			(show_name no)
+			(do_not_autoplace no)
+			(effects
+				(font
+					(size 1.27 1.27)
+				)
+			)
+		)
+		(property "FT Layer Override" "bottom"
+			(at 125.73 96.52 0)
+			(hide yes)
+			(show_name no)
+			(do_not_autoplace no)
+			(effects
+				(font
+					(size 1.27 1.27)
+				)
+			)
+		)
+		(property "FT Rotation Offset" "180"
+			(at 125.73 96.52 0)
+			(hide yes)
+			(show_name no)
+			(do_not_autoplace no)
+			(effects
+				(font
+					(size 1.27 1.27)
+				)
+			)
+		)
+		(property "FT Position Offset" "0.635,3.81"
+			(at 125.73 96.52 0)
+			(hide yes)
