File: keyboard/key.kicad_sch (KiCad schematic)
At the start: 4 parts, among them SW2 MX

Commit message: ISO version of the keyboard
Parts:
- D2: footprint LED_SMD:LED_SK6812MINI-E_3.2x2.8mm_P1.5mm_ReverseMount -> Library:LED_SK6812MINI-E_3.2x2.8mm_P1.5mm_ReverseMount
- SW2: footprint Library:SMD_KEYBOARD-SW -> Library:Kailh_socket_MX_1-00U
Connections:
- net GND: now also D2.1 (VSS); no longer D2.3 (VSS)
- net RGB_IN: now also D2.2 (DIN); no longer D2.4 (DIN)
- net RGB_OUT: now also D2.4 (DOUT); no longer D2.2 (DOUT)
- net VBUS renamed VSYS
- net VSYS: now also D2.3 (VDD); no longer D2.1 (VDD)
