File: keyboard/rgb.kicad_sch (KiCad schematic)
At the start: 2 parts

Commit message: Production file fixes for the keyboard PCB
Parts:
- D149: FT Rotation Offset (none) -> 180; LCSC Part # C5149201 -> C5378731
Changed lines of the file:
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@@
 			)
 		)
-		(property "LCSC Part #" "C5149201"
+		(property "LCSC Part #" "C5378731"
 			(at 132.08 91.44 0)
 			(hide yes)
@@
 		)
 		(property "FT Origin" ""
+			(at 132.08 91.44 0)
+			(hide yes)
+			(show_name no)
+			(do_not_autoplace no)
+			(effects
+				(font
+					(size 1.27 1.27)
+				)
+			)
+		)
+		(property "FT Layer Override" ""
+			(at 132.08 91.44 0)
+			(hide yes)
+			(show_name no)
+			(do_not_autoplace no)
+			(effects
+				(font
+					(size 1.27 1.27)
+				)
+			)
+		)
+		(property "FT Rotation Offset" "180"
 			(at 132.08 91.44 0)
 			(hide yes)
@@
 			(at 153.67 91.44 0)
 			(hide yes)
+			(show_name no)
+			(do_not_autoplace no)
+			(effects
+				(font
+					(size 1.27 1.27)
+				)
+			)
+		)
+		(property "FT Layer Override" ""
+			(at 153.67 91.44 0)
+			(hide yes)
