File: keyboard/controller.kicad_sch (KiCad schematic)
At the start: 37 parts, among them J1 Conn_01x04_Socket, J4 Conn_01x04_Pin, J5 USB_C_Receptacle_USB2.0_16P, J6 Conn_01x04, J9 SM03B-SRSS-TB, SW2 SW_BOOT_SELECT, SW3 SW_RESET, U4 NCP1117-3.3, U7 RP2040, U9 W25Q128JVS, X1 12MHz

Commit message: ISO version of the keyboard
Parts:
- renumbered C43 to C78, C42 to C79, C27 to C80, C28 to C81, C24 to C82, C25 to C83, C4 to C84, C5 to C85, C6 to C86, C7 to C87, C8 to C88, C9 to C89, C10 to C90, C11 to C91, C12 to C92, C13 to C93, C14 to C94, J5 to J1, J4 to J2, J9 to J3, J6 to J4, J1 to J5, R37 to R1, R36 to R2, R7 to R3, R6 to R4, R30 to R5, R31 to R6, R26 to R7, R28 to R8, R32 to R9, SW2 to SW68, SW3 to SW69, U9 to U1, U4 to U2, U7 to U3
